File: ECE-445-Chess-Board/ECE-445-Chess-Board.kicad_sch (KiCad schematic)
At the start: 0 parts

Commit message: added hall sensors and started ADC schematic
Other:
- added sheet ADC_Suite (ADC_Suite.kicad_sch)
Changed lines of the file:
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@@
 	(generator_version "9.0")
 	(paper "A4")
+	(sheet
+		(at 44.45 77.47)
+		(size 12.7 15.24)
+		(exclude_from_sim no)
+		(in_bom yes)
+		(on_board yes)
+		(dnp no)
+		(fields_autoplaced yes)
+		(stroke
+			(width 0.1524)
+			(type solid)
+		)
+		(fill
+			(color 0 0 0 0.0000)
+		)
+		(property "Sheetname" "ADC_Suite"
+			(at 44.45 76.7584 0)
+			(effects
+				(font
+					(size 1.27 1.27)
+				)
+				(justify left bottom)
+			)
+		)
+		(property "Sheetfile" "ADC_Suite.kicad_sch"
+			(at 44.45 93.2946 0)
+			(effects
+				(font
+					(size 1.27 1.27)
+				)
+				(justify left top)
+			)
+		)
+		(instances
+			(project "ECE-445-Chess-Board"
+				(path "/7211742c-a67f-4955-9f8b-c5c6ecfe8b63"
+					(page "3")
+				)
+			)
+		)
+	)
 	(sheet_instances
 		(path "/"
