File: ECE-445-PCBs/Main_Board/Main_Board_PCB.kicad_pcb (KiCad board)
At the start: 2 copper layers, 100 x 100 mm, 20 parts, among them J1 USB_C_Receptacle_USB2.0_16P, J10 Conn_02x05_Odd_Even, J11 Conn_02x05_Odd_Even, J2 Screw_Terminal_01x08, J3 Conn_01x02_Pin, J4 Conn_02x05_Odd_Even, J5 Conn_02x05_Odd_Even, J6 Conn_02x05_Odd_Even, J7 Conn_02x05_Odd_Even, J8 Conn_02x05_Odd_Even, J9 Conn_02x05_Odd_Even, U1 ESP32-S3-WROOM-1, U2 TLV62569DDC, U3 ADS7128IRTER, U4 ADS7128IRTER, U5 ADS7128IRTER, U6 ADS7128IRTER, U7 ADS7128IRTER, U8 ADS7128IRTER, U9 ADS7128IRTER

Commit message: started placement
Parts:
- removed the J4 at (126.5, 115.3)
- added C1: 1uF, Capacitor_SMD:C_0603_1608Metric, F.Cu at (219.7, 85.7)
- added C10: 0.1uF, Capacitor_SMD:C_0603_1608Metric, F.Cu at (172.7, 63.5)
- added C11: 1uF, Capacitor_SMD:C_0603_1608Metric, F.Cu at (207.9, 125.0)
- added C12: 1uF, Capacitor_SMD:C_0603_1608Metric, F.Cu at (207.9, 127.5)
- added C13: 1uF, Capacitor_SMD:C_0603_1608Metric, F.Cu at (207.9, 130.0)
- added C14: 10uF, Capacitor_SMD:C_0603_1608Metric, F.Cu at (207.9, 137.1)
- added C15: 0.1uF, Capacitor_SMD:C_0603_1608Metric, F.Cu at (207.9, 139.6)
- added C16: 1uF, Capacitor_SMD:C_0603_1608Metric, F.Cu at (207.9, 142.1)
- added C17: 1uF, Capacitor_SMD:C_0603_1608Metric, F.Cu at (207.9, 144.6)
- added C18: 1uF, Capacitor_SMD:C_0603_1608Metric, F.Cu at (207.9, 147.1)
- added C19: 10uF, Capacitor_SMD:C_0603_1608Metric, F.Cu at (228.8, 120.0)
- added C2: 1uF, Capacitor_SMD:C_0603_1608Metric, F.Cu at (219.7, 88.2)
- added C20: 0.1uF, Capacitor_SMD:C_0603_1608Metric, F.Cu at (228.8, 122.5)
- added C21: 1uF, Capacitor_SMD:C_0603_1608Metric, F.Cu at (228.8, 125.0)
- added C22: 1uF, Capacitor_SMD:C_0603_1608Metric, F.Cu at (228.8, 127.5)
- added C23: 1uF, Capacitor_SMD:C_0603_1608Metric, F.Cu at (228.8, 130.0)
- added C24: 10uF, Capacitor_SMD:C_0603_1608Metric, F.Cu at (249.6, 120.0)
- added C25: 0.1uF, Capacitor_SMD:C_0603_1608Metric, F.Cu at (249.6, 122.5)
- added C26: 1uF, Capacitor_SMD:C_0603_1608Metric, F.Cu at (249.6, 125.0)
- added C27: 1uF, Capacitor_SMD:C_0603_1608Metric, F.Cu at (249.6, 127.5)
- added C28: 1uF, Capacitor_SMD:C_0603_1608Metric, F.Cu at (249.6, 130.0)
- added C29: 10uF, Capacitor_SMD:C_0603_1608Metric, F.Cu at (247.5, 95.6)
- added C3: 4.7uF, Capacitor_SMD:C_0603_1608Metric, F.Cu at (219.7, 90.7)
- added C30: 0.1uF, Capacitor_SMD:C_0603_1608Metric, F.Cu at (247.5, 98.1)
- added C31: 1uF, Capacitor_SMD:C_0603_1608Metric, F.Cu at (247.5, 100.6)
- added C32: 1uF, Capacitor_SMD:C_0603_1608Metric, F.Cu at (247.5, 103.1)
- added C33: 1uF, Capacitor_SMD:C_0603_1608Metric, F.Cu at (247.5, 105.6)
- added C34: 10uF, Capacitor_SMD:C_0603_1608Metric, F.Cu at (228.8, 137.1)
- added C35: 0.1uF, Capacitor_SMD:C_0603_1608Metric, F.Cu at (228.8, 139.6)
- added C36: 1uF, Capacitor_SMD:C_0603_1608Metric, F.Cu at (228.8, 142.1)
- added C37: 1uF, Capacitor_SMD:C_0603_1608Metric, F.Cu at (228.8, 144.6)
- added C38: 1uF, Capacitor_SMD:C_0603_1608Metric, F.Cu at (228.8, 147.1)
- added C39: 10uF, Capacitor_SMD:C_0603_1608Metric, F.Cu at (249.6, 137.1)
- added C4: 10uF, Capacitor_SMD:C_0603_1608Metric, F.Cu at (219.7, 93.2)
- added C40: 0.1uF, Capacitor_SMD:C_0603_1608Metric, F.Cu at (249.6, 139.6)
- added C41: 1uF, Capacitor_SMD:C_0603_1608Metric, F.Cu at (249.6, 142.1)
- added C42: 1uF, Capacitor_SMD:C_0603_1608Metric, F.Cu at (249.6, 144.6)
- added C43: 1uF, Capacitor_SMD:C_0603_1608Metric, F.Cu at (249.6, 147.1)
- added C44: 10uF, Capacitor_SMD:C_0603_1608Metric, F.Cu at (247.5, 78.5)
- added C45: 0.1uF, Capacitor_SMD:C_0603_1608Metric, F.Cu at (247.5, 81.0)
- added C46: 1uF, Capacitor_SMD:C_0603_1608Metric, F.Cu at (247.5, 83.6)
- added C47: 1uF, Capacitor_SMD:C_0603_1608Metric, F.Cu at (247.5, 86.1)
- added C48: 1uF, Capacitor_SMD:C_0603_1608Metric, F.Cu at (247.5, 88.6)
- added C5: 10uF, Capacitor_SMD:C_0603_1608Metric, F.Cu at (219.7, 95.7)
- added C6: 22uF, Capacitor_SMD:C_0603_1608Metric, F.Cu at (219.7, 98.2)
- added C7: 10uF, Capacitor_SMD:C_0603_1608Metric, F.Cu at (219.7, 100.7)
- added C8: 0.1uF, Capacitor_SMD:C_0603_1608Metric, F.Cu at (223.7, 85.7)
- added C9: 10uF, Capacitor_SMD:C_0603_1608Metric, F.Cu at (174.2, 63.5)
- added D1: RED LED, LED_SMD:LED_0603_1608Metric, F.Cu at (229.2, 107.1)
- added D2: RED LED, LED_SMD:LED_0603_1608Metric, F.Cu at (229.2, 109.7)
- added H1: MountingHole_Pad, MountingHole:MountingHole_3.2mm_M3_DIN965_Pad, F.Cu at (187.8, 56.5)
- added H2: MountingHole_Pad, MountingHole:MountingHole_3.2mm_M3_DIN965_Pad, F.Cu at (95.8, 56.5)
- added H3: MountingHole_Pad, MountingHole:MountingHole_3.2mm_M3_DIN965_Pad, F.Cu at (95.8, 142.2)
- added H4: MountingHole_Pad, MountingHole:MountingHole_3.2mm_M3_DIN965_Pad, F.Cu at (187.8, 142.2)
- added J1: Conn_01x14_Pin, Connector_PinHeader_2.54mm:PinHeader_1x14_P2.54mm_Vertical, F.Cu at (212.5, 79.5)
- added J12: Conn_02x05_Odd_Even, Connector_Amphenol:AMPHENOL_67997-410HLF, F.Cu at (181.7, 85.5)
- added J13: Conn_02x05_Odd_Even, Connector_Amphenol:AMPHENOL_67997-410HLF, F.Cu at (181.7, 91.0)
- added J14: Conn_02x05_Odd_Even, Connector_Amphenol:AMPHENOL_67997-410HLF, F.Cu at (181.7, 96.5)
- added J15: Conn_02x05_Odd_Even, Connector_Amphenol:AMPHENOL_67997-410HLF, F.Cu at (181.7, 102.0)
- added JP1: SolderJumper_3_Open, Jumper:SolderJumper-3_P1.3mm_Open_Pad1.0x1.5mm, F.Cu at (230.0, 103.8)
- added JP2: SolderJumper_2_Open, Jumper:SolderJumper-2_P1.3mm_Open_Pad1.0x1.5mm, F.Cu at (233.4, 112.2)
- added L1: 2.2uH, Inductor_SMD:L_Coilcraft_1008HQ_2520Metric, F.Cu at (233.7, 108.2)
- added Q1: SS8050, Package_TO_SOT_SMD:SOT-23, F.Cu at (224.7, 104.2)
- added Q2: SS8050, Package_TO_SOT_SMD:SOT-23, F.Cu at (224.7, 108.7)
- added R1: 100k, Resistor_SMD:R_0603_1608Metric, F.Cu at (223.7, 88.2)
- added R10: 5.1k, Resistor_SMD:R_0603_1608Metric, F.Cu at (227.7, 93.2)
- added R11: 10k, Resistor_SMD:R_0603_1608Metric, F.Cu at (227.7, 95.7)
- added R12: 10k, Resistor_SMD:R_0603_1608Metric, F.Cu at (227.7, 98.2)
- added R13: 475k, Resistor_SMD:R_0603_1608Metric, F.Cu at (227.7, 100.7)
- added R14: 450k, Resistor_SMD:R_0603_1608Metric, F.Cu at (231.7, 85.7)
- added R15: 100k, Resistor_SMD:R_0603_1608Metric, F.Cu at (231.7, 88.2)
- added R16: 1k, Resistor_SMD:R_0603_1608Metric, F.Cu at (231.7, 90.7)
- added R17: 470, Resistor_SMD:R_0603_1608Metric, F.Cu at (231.7, 93.2)
- added R18: 470, Resistor_SMD:R_0603_1608Metric, F.Cu at (231.7, 95.7)
- added R19: 1k, Resistor_SMD:R_0603_1608Metric, F.Cu at (231.7, 98.2)
- added R2: 4.7k, Resistor_SMD:R_0603_1608Metric, F.Cu at (223.7, 90.7)
- added R20: 4.7k, Resistor_SMD:R_0603_1608Metric, F.Cu at (207.9, 132.6)
- added R21: 4.7k, Resistor_SMD:R_0603_1608Metric, F.Cu at (207.9, 149.6)
- added R22: 4.7k, Resistor_SMD:R_0603_1608Metric, F.Cu at (228.8, 132.6)
- added R23: 4.7k, Resistor_SMD:R_0603_1608Metric, F.Cu at (249.6, 132.6)
- added R24: 4.7k, Resistor_SMD:R_0603_1608Metric, F.Cu at (247.5, 108.2)
- added R25: 4.7k, Resistor_SMD:R_0603_1608Metric, F.Cu at (228.8, 149.6)
- added R26: 4.7k, Resistor_SMD:R_0603_1608Metric, F.Cu at (249.6, 149.6)
- added R27: 4.7k, Resistor_SMD:R_0603_1608Metric, F.Cu at (247.5, 91.1)
- added R28: 0, Resistor_SMD:R_0603_1608Metric, F.Cu at (268.3, 95.6)
- added R29: R_US, Resistor_SMD:R_0603_1608Metric, F.Cu at (268.3, 98.1)
- added R3: 4.7k, Resistor_SMD:R_0603_1608Metric, F.Cu at (223.7, 93.2)
- added R30: 11k, Resistor_SMD:R_0603_1608Metric, F.Cu at (268.3, 100.6)
- added R31: R_US, Resistor_SMD:R_0603_1608Metric, F.Cu at (268.3, 103.1)
- added R32: 33k, Resistor_SMD:R_0603_1608Metric, F.Cu at (268.3, 105.6)
- added R33: R_US, Resistor_SMD:R_0603_1608Metric, F.Cu at (268.3, 108.2)
- added R34: 100k, Resistor_SMD:R_0603_1608Metric, F.Cu at (272.3, 95.6)
- added R35: R_US, Resistor_SMD:R_0603_1608Metric, F.Cu at (272.3, 98.1)
- added R36: R_US, Resistor_SMD:R_0603_1608Metric, F.Cu at (272.3, 100.6)
- added R37: R_US, Resistor_SMD:R_0603_1608Metric, F.Cu at (272.3, 103.1)
- added R38: R_US, Resistor_SMD:R_0603_1608Metric, F.Cu at (272.3, 105.6)
- added R39: 11k, Resistor_SMD:R_0603_1608Metric, F.Cu at (272.3, 108.2)
- added R4: 100k, Resistor_SMD:R_0603_1608Metric, F.Cu at (223.7, 95.7)
- added R40: R_US, Resistor_SMD:R_0603_1608Metric, F.Cu at (276.3, 95.6)
- added R41: 33k, Resistor_SMD:R_0603_1608Metric, F.Cu at (276.3, 98.1)
- added R42: R_US, Resistor_SMD:R_0603_1608Metric, F.Cu at (276.3, 100.6)
- added R43: 100k, Resistor_SMD:R_0603_1608Metric, F.Cu at (276.3, 103.1)
- added R5: 4.7k, Resistor_SMD:R_0603_1608Metric, F.Cu at (223.7, 98.2)
- added R6: 4.7k, Resistor_SMD:R_0603_1608Metric, F.Cu at (223.7, 100.7)
- added R7: 10k, Resistor_SMD:R_0603_1608Metric, F.Cu at (227.7, 85.7)
- added R8: 10k, Resistor_SMD:R_0603_1608Metric, F.Cu at (227.7, 88.2)
- added R9: 5.1k, Resistor_SMD:R_0603_1608Metric, F.Cu at (227.7, 90.7)
- added SW1: SW_Push, Button_Switch_THT:SW_TH_Tactile_Omron_B3F-100x, F.Cu at (235.3, 85.5)
- added SW2: SW_Push, Button_Switch_THT:SW_TH_Tactile_Omron_B3F-100x, F.Cu at (235.3, 93.8)
- added U10: ADS7128IRTER, Package_DFN_QFN:WQFN16_RTE_TEX-M, F.Cu at (252.5, 86.7)
- J2: value Screw_Terminal_01x08 -> Conn_01x02_Pin; footprint TerminalBlock:OSTVN08A150 -> Connector_PinHeader_2.54mm:PinHeader_1x02_P2.54mm_Vertical
- J3: footprint Connector_Harwin:HARWIN_M20-9990246 -> Connector_PinHeader_2.54mm:PinHeader_1x02_P2.54mm_Vertical
- J4: renamed from J1; footprint Connector_USB:USB4215-03-A -> Connector_USB:USB_C_Receptacle_G-Switch_GT-USB-7010ASV
- J5, J6: value Conn_02x05_Odd_Even -> Conn_01x02_Pin; footprint Connector_Amphenol:AMPHENOL_67997-410HLF -> Connector_PinHeader_2.54mm:PinHeader_1x02_P2.54mm_Vertical
- J7: value Conn_02x05_Odd_Even -> Conn_01x05_Pin; footprint Connector_Amphenol:AMPHENOL_67997-410HLF -> Connector_PinHeader_2.54mm:PinHeader_1x05_P2.54mm_Vertical
- moved J2 102.0 mm to (220.0, 79.6)
- moved J6 96.8 mm to (233.7, 79.6)
- moved U6 94.7 mm to (254.7, 128.2)
- moved U9 90.2 mm to (254.7, 145.3)
- moved J5 89.7 mm to (229.2, 79.6)
- moved U7 87.1 mm to (252.5, 103.8)
- moved J11 86.1 mm to (181.7, 80.0), turned to 180 degrees
- moved J10 85.2 mm to (181.7, 74.5), turned to 180 degrees
- moved J9 84.4 mm to (181.7, 69.0), turned to 180 degrees
- moved J8 83.6 mm to (181.7, 63.5), turned to 180 degrees
- moved J7 76.3 mm to (220.0, 104.3)
- moved U1 74.7 mm to (213.0, 58.2)
- moved U5 73.7 mm to (233.8, 128.2)
- moved J3 72.4 mm to (224.6, 79.6)
- moved U8 71.7 mm to (233.8, 145.3)
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- renumbered U2 to U1, U1 to U2
Connections:
- J10 pad 1: unconnected-(J10-Pin_1-Pad1) -> /ADC_Group/Hall_Effect_Acquisition2/HE_Sensor_0
- J10 pad 10: unconnected-(J10-Pin_10-Pad10) -> GND
- J10 pad 2: unconnected-(J10-Pin_2-Pad2) -> /ADC_Group/Hall_Effect_Acquisition2/HE_Sensor_1
- J10 pad 3: unconnected-(J10-Pin_3-Pad3) -> /ADC_Group/Hall_Effect_Acquisition2/HE_Sensor_2
- J10 pad 4: unconnected-(J10-Pin_4-Pad4) -> /ADC_Group/Hall_Effect_Acquisition2/HE_Sensor_3
- J10 pad 5: unconnected-(J10-Pin_5-Pad5) -> /ADC_Group/Hall_Effect_Acquisition2/HE_Sensor_4
- J10 pad 6: unconnected-(J10-Pin_6-Pad6) -> /ADC_Group/Hall_Effect_Acquisition2/HE_Sensor_5
- J10 pad 7: unconnected-(J10-Pin_7-Pad7) -> /ADC_Group/Hall_Effect_Acquisition2/HE_Sensor_6
- J10 pad 8: unconnected-(J10-Pin_8-Pad8) -> /ADC_Group/Hall_Effect_Acquisition2/HE_Sensor_7
- J10 pad 9: unconnected-(J10-Pin_9-Pad9) -> /ADC_Group/Hall_Effect_Acquisition2/3V3
- J11 pad 1: unconnected-(J11-Pin_1-Pad1) -> /ADC_Group/Hall_Effect_Acquisition3/HE_Sensor_0
- J11 pad 10: unconnected-(J11-Pin_10-Pad10) -> GND
- J11 pad 2: unconnected-(J11-Pin_2-Pad2) -> /ADC_Group/Hall_Effect_Acquisition3/HE_Sensor_1
- J11 pad 3: unconnected-(J11-Pin_3-Pad3) -> /ADC_Group/Hall_Effect_Acquisition3/HE_Sensor_2
- J11 pad 4: unconnected-(J11-Pin_4-Pad4) -> /ADC_Group/Hall_Effect_Acquisition3/HE_Sensor_3
- J11 pad 5: unconnected-(J11-Pin_5-Pad5) -> /ADC_Group/Hall_Effect_Acquisition3/HE_Sensor_4
- J11 pad 6: unconnected-(J11-Pin_6-Pad6) -> /ADC_Group/Hall_Effect_Acquisition3/HE_Sensor_5
- J11 pad 7: unconnected-(J11-Pin_7-Pad7) -> /ADC_Group/Hall_Effect_Acquisition3/HE_Sensor_6
- J11 pad 8: unconnected-(J11-Pin_8-Pad8) -> /ADC_Group/Hall_Effect_Acquisition3/HE_Sensor_7
- J11 pad 9: unconnected-(J11-Pin_9-Pad9) -> /ADC_Group/Hall_Effect_Acquisition3/3V3
- J2 pad 1: unconnected-(J2-Pin_1-Pad1) -> /I2C_SDA_DAQ
- J2 pad 2: unconnected-(J2-Pin_2-Pad2) -> /I2C_SCL_DAQ
- J3 pad 1: unconnected-(J3-Pin_1-Pad1) -> /I2C_SCL_SCR
- J3 pad 2: unconnected-(J3-Pin_2-Pad2) -> /I2C_SDA_SCR
- J4 pad A5: unconnected-(J1-CC1-PadA5) -> Net-(J4-CC1)
- J4 pad A6: unconnected-(J1-D+-PadA6) -> /USB_D_P
- J4 pad A7: unconnected-(J1-D--PadA7) -> /USB_D_N
- J4 pad B5: unconnected-(J1-CC2-PadB5) -> Net-(J4-CC2)
- J4 pad B6: unconnected-(J1-D+-PadB6) -> /USB_D_P
- J4 pad B7: unconnected-(J1-D--PadB7) -> /USB_D_N
- J5 pad 1: unconnected-(J5-Pin_1-Pad1) -> /5V
- J5 pad 2: unconnected-(J5-Pin_2-Pad2) -> GND
- J6 pad 1: unconnected-(J6-Pin_1-Pad1) -> /3V3
- J6 pad 2: unconnected-(J6-Pin_2-Pad2) -> GND
- J7 pad 1: unconnected-(J7-Pin_1-Pad1) -> /RTS
- J7 pad 2: unconnected-(J7-Pin_2-Pad2) -> /DTR
- J7 pad 3: unconnected-(J7-Pin_3-Pad3) -> /TX
- J7 pad 4: unconnected-(J7-Pin_4-Pad4) -> /RX
- J7 pad 5: unconnected-(J7-Pin_5-Pad5) -> GND
- J8 pad 1: unconnected-(J8-Pin_1-Pad1) -> /ADC_Group/Hall_Effect_Acquisition/HE_Sensor_0
- J8 pad 10: unconnected-(J8-Pin_10-Pad10) -> GND
- J8 pad 2: unconnected-(J8-Pin_2-Pad2) -> /ADC_Group/Hall_Effect_Acquisition/HE_Sensor_1
- J8 pad 3: unconnected-(J8-Pin_3-Pad3) -> /ADC_Group/Hall_Effect_Acquisition/HE_Sensor_2
- J8 pad 4: unconnected-(J8-Pin_4-Pad4) -> /ADC_Group/Hall_Effect_Acquisition/HE_Sensor_3
- J8 pad 5: unconnected-(J8-Pin_5-Pad5) -> /ADC_Group/Hall_Effect_Acquisition/HE_Sensor_4
- J8 pad 6: unconnected-(J8-Pin_6-Pad6) -> /ADC_Group/Hall_Effect_Acquisition/HE_Sensor_5
- J8 pad 7: unconnected-(J8-Pin_7-Pad7) -> /ADC_Group/Hall_Effect_Acquisition/HE_Sensor_6
- J8 pad 8: unconnected-(J8-Pin_8-Pad8) -> /ADC_Group/Hall_Effect_Acquisition/HE_Sensor_7
- J8 pad 9: unconnected-(J8-Pin_9-Pad9) -> /ADC_Group/Hall_Effect_Acquisition/3V3
- J9 pad 1: unconnected-(J9-Pin_1-Pad1) -> /ADC_Group/Hall_Effect_Acquisition1/HE_Sensor_0
- J9 pad 10: unconnected-(J9-Pin_10-Pad10) -> GND
- J9 pad 2: unconnected-(J9-Pin_2-Pad2) -> /ADC_Group/Hall_Effect_Acquisition1/HE_Sensor_1
- J9 pad 3: unconnected-(J9-Pin_3-Pad3) -> /ADC_Group/Hall_Effect_Acquisition1/HE_Sensor_2
- J9 pad 4: unconnected-(J9-Pin_4-Pad4) -> /ADC_Group/Hall_Effect_Acquisition1/HE_Sensor_3
- J9 pad 5: unconnected-(J9-Pin_5-Pad5) -> /ADC_Group/Hall_Effect_Acquisition1/HE_Sensor_4
- J9 pad 6: unconnected-(J9-Pin_6-Pad6) -> /ADC_Group/Hall_Effect_Acquisition1/HE_Sensor_5
- J9 pad 7: unconnected-(J9-Pin_7-Pad7) -> /ADC_Group/Hall_Effect_Acquisition1/HE_Sensor_6
- J9 pad 8: unconnected-(J9-Pin_8-Pad8) -> /ADC_Group/Hall_Effect_Acquisition1/HE_Sensor_7
- J9 pad 9: unconnected-(J9-Pin_9-Pad9) -> /ADC_Group/Hall_Effect_Acquisition1/3V3
- U1 pad 1: unconnected-(U2-EN-Pad1) -> /5V
- U1 pad 2: unconnected-(U2-GND-Pad2) -> GND
- U1 pad 3: unconnected-(U2-SW-Pad3) -> Net-(U1-SW)
- U1 pad 4: unconnected-(U2-VIN-Pad4) -> /5V
- U1 pad 5: unconnected-(U2-PG-Pad5) -> Net-(U1-PG)
- U1 pad 6: unconnected-(U2-FB-Pad6) -> Net-(U1-FB)
- U2 pad 1: Net-(U1-GND-Pad1) -> GND
- U2 pad 10: unconnected-(U1-IO17-Pad10) -> /SCR_DC
- U2 pad 11: unconnected-(U1-IO18-Pad11) -> /SCR_BLK
- U2 pad 12: unconnected-(U1-IO8-Pad12) -> /ADC4_ALERT
- U2 pad 13: unconnected-(U1-USB_D--Pad13) -> /USB_D_N
- U2 pad 14: unconnected-(U1-USB_D+-Pad14) -> /USB_D_P
- U2 pad 15: unconnected-(U1-IO3-Pad15) -> Net-(U2-IO3)
- U2 pad 16: unconnected-(U1-IO46-Pad16) -> Net-(U2-IO46)
- U2 pad 17: unconnected-(U1-IO9-Pad17) -> /ADC5_ALERT
- U2 pad 18: unconnected-(U1-IO10-Pad18) -> /ADC6_ALERT
- U2 pad 19: unconnected-(U1-IO11-Pad19) -> /ADC7_ALERT
- U2 pad 2: unconnected-(U1-3V3-Pad2) -> /3V3
- U2 pad 20: unconnected-(U1-IO12-Pad20) -> /I2C_SCL_DAQ
- U2 pad 21: unconnected-(U1-IO13-Pad21) -> /I2C_SDA_DAQ
- U2 pad 22: unconnected-(U1-IO14-Pad22) -> /I2C_SCL_SCR
- U2 pad 23: unconnected-(U1-IO21-Pad23) -> /SCR_INT
- U2 pad 25: unconnected-(U1-IO48-Pad25) -> Net-(U2-IO48)
- U2 pad 27: unconnected-(U1-IO0-Pad27) -> /ESP_BOOT
- U2 pad 3: unconnected-(U1-EN-Pad3) -> /ESP_EN
- U2 pad 31: unconnected-(U1-IO38-Pad31) -> /SCR_SCLK
- U2 pad 32: unconnected-(U1-IO39-Pad32) -> /SCR_MOSI
- U2 pad 33: unconnected-(U1-IO40-Pad33) -> /SCR_MISO
- U2 pad 34: unconnected-(U1-IO41-Pad34) -> /SCR_CS
- U2 pad 36: unconnected-(U1-RXD0-Pad36) -> /RX
- U2 pad 37: unconnected-(U1-TXD0-Pad37) -> /TX
- U2 pad 38: unconnected-(U1-IO2-Pad38) -> /TCH_RST
- U2 pad 39: unconnected-(U1-IO1-Pad39) -> /SCR_RST
- U2 pad 4: unconnected-(U1-IO4-Pad4) -> /ADC0_ALERT
- U2 pad 40: Net-(U1-GND-Pad1) -> GND
- U2 pad 41: Net-(U1-GND-Pad1) -> GND
- U2 pad 5: unconnected-(U1-IO5-Pad5) -> /ADC1_ALERT
- U2 pad 6: unconnected-(U1-IO6-Pad6) -> /ADC2_ALERT
- U2 pad 7: unconnected-(U1-IO7-Pad7) -> /ADC3_ALERT
- U2 pad 8: unconnected-(U1-IO15-Pad8) -> /I2C_SDA_SCR
- U3 pad 1: unconnected-(U3-AIN2/GPIO2-Pad1) -> /ADC_Group/Hall_Effect_Acquisition/HE_Sensor_2
- U3 pad 10: unconnected-(U3-DVDD-Pad10) -> /ADC_Group/Hall_Effect_Acquisition/3V3
- U3 pad 11: unconnected-(U3-ADDR-Pad11) -> /ADC_Group/Hall_Effect_Acquisition/ADC_ADDR
- U3 pad 12: unconnected-(U3-ALERT-Pad12) -> /ADC0_ALERT
- U3 pad 13: unconnected-(U3-SCL-Pad13) -> /I2C_SCL_DAQ
- U3 pad 14: unconnected-(U3-SDA-Pad14) -> /I2C_SDA_DAQ
- U3 pad 15: unconnected-(U3-AIN0/GPIO0-Pad15) -> /ADC_Group/Hall_Effect_Acquisition/HE_Sensor_0
- U3 pad 16: unconnected-(U3-AIN1/GPIO1-Pad16) -> /ADC_Group/Hall_Effect_Acquisition/HE_Sensor_1
- U3 pad 17: unconnected-(U3-GND-Pad17) -> GND
- U3 pad 2: unconnected-(U3-AIN3/GPIO3-Pad2) -> /ADC_Group/Hall_Effect_Acquisition/HE_Sensor_3
- U3 pad 3: unconnected-(U3-AIN4/GPIO4-Pad3) -> /ADC_Group/Hall_Effect_Acquisition/HE_Sensor_4
- U3 pad 4: unconnected-(U3-AIN5/GPIO5-Pad4) -> /ADC_Group/Hall_Effect_Acquisition/HE_Sensor_5
- U3 pad 5: unconnected-(U3-AIN6/GPIO6-Pad5) -> /ADC_Group/Hall_Effect_Acquisition/HE_Sensor_6
- U3 pad 6: unconnected-(U3-AIN7/GPIO7-Pad6) -> /ADC_Group/Hall_Effect_Acquisition/HE_Sensor_7
- U3 pad 7: unconnected-(U3-AVDD-Pad7) -> /ADC_Group/Hall_Effect_Acquisition/3V3
- U3 pad 8: unconnected-(U3-DECAP-Pad8) -> /ADC_Group/Hall_Effect_Acquisition/Decap
- U3 pad 9: unconnected-(U3-GND-Pad9) -> GND
- U4 pad 1: unconnected-(U4-AIN2/GPIO2-Pad1) -> /ADC_Group/Hall_Effect_Acquisition1/HE_Sensor_2
- U4 pad 10: unconnected-(U4-DVDD-Pad10) -> /ADC_Group/Hall_Effect_Acquisition1/3V3
- U4 pad 11: unconnected-(U4-ADDR-Pad11) -> /ADC_Group/Hall_Effect_Acquisition1/ADC_ADDR
- U4 pad 12: unconnected-(U4-ALERT-Pad12) -> /ADC1_ALERT
- U4 pad 13: unconnected-(U4-SCL-Pad13) -> /I2C_SCL_DAQ
- U4 pad 14: unconnected-(U4-SDA-Pad14) -> /I2C_SDA_DAQ
- U4 pad 15: unconnected-(U4-AIN0/GPIO0-Pad15) -> /ADC_Group/Hall_Effect_Acquisition1/HE_Sensor_0
- U4 pad 16: unconnected-(U4-AIN1/GPIO1-Pad16) -> /ADC_Group/Hall_Effect_Acquisition1/HE_Sensor_1
- U4 pad 17: unconnected-(U4-GND-Pad17) -> GND
- U4 pad 2: unconnected-(U4-AIN3/GPIO3-Pad2) -> /ADC_Group/Hall_Effect_Acquisition1/HE_Sensor_3
- U4 pad 3: unconnected-(U4-AIN4/GPIO4-Pad3) -> /ADC_Group/Hall_Effect_Acquisition1/HE_Sensor_4
- U4 pad 4: unconnected-(U4-AIN5/GPIO5-Pad4) -> /ADC_Group/Hall_Effect_Acquisition1/HE_Sensor_5
- U4 pad 5: unconnected-(U4-AIN6/GPIO6-Pad5) -> /ADC_Group/Hall_Effect_Acquisition1/HE_Sensor_6
- U4 pad 6: unconnected-(U4-AIN7/GPIO7-Pad6) -> /ADC_Group/Hall_Effect_Acquisition1/HE_Sensor_7
- U4 pad 7: unconnected-(U4-AVDD-Pad7) -> /ADC_Group/Hall_Effect_Acquisition1/3V3
- U4 pad 8: unconnected-(U4-DECAP-Pad8) -> /ADC_Group/Hall_Effect_Acquisition1/Decap
- U4 pad 9: unconnected-(U4-GND-Pad9) -> GND
- U5 pad 1: unconnected-(U5-AIN2/GPIO2-Pad1) -> /ADC_Group/Hall_Effect_Acquisition2/HE_Sensor_2
- U5 pad 10: unconnected-(U5-DVDD-Pad10) -> /ADC_Group/Hall_Effect_Acquisition2/3V3
- U5 pad 11: unconnected-(U5-ADDR-Pad11) -> /ADC_Group/Hall_Effect_Acquisition2/ADC_ADDR
- U5 pad 12: unconnected-(U5-ALERT-Pad12) -> /ADC2_ALERT
- U5 pad 13: unconnected-(U5-SCL-Pad13) -> /I2C_SCL_DAQ
- U5 pad 14: unconnected-(U5-SDA-Pad14) -> /I2C_SDA_DAQ
- U5 pad 15: unconnected-(U5-AIN0/GPIO0-Pad15) -> /ADC_Group/Hall_Effect_Acquisition2/HE_Sensor_0
- U5 pad 16: unconnected-(U5-AIN1/GPIO1-Pad16) -> /ADC_Group/Hall_Effect_Acquisition2/HE_Sensor_1
- U5 pad 17: unconnected-(U5-GND-Pad17) -> GND
- U5 pad 2: unconnected-(U5-AIN3/GPIO3-Pad2) -> /ADC_Group/Hall_Effect_Acquisition2/HE_Sensor_3
- U5 pad 3: unconnected-(U5-AIN4/GPIO4-Pad3) -> /ADC_Group/Hall_Effect_Acquisition2/HE_Sensor_4
- U5 pad 4: unconnected-(U5-AIN5/GPIO5-Pad4) -> /ADC_Group/Hall_Effect_Acquisition2/HE_Sensor_5
- U5 pad 5: unconnected-(U5-AIN6/GPIO6-Pad5) -> /ADC_Group/Hall_Effect_Acquisition2/HE_Sensor_6
- U5 pad 6: unconnected-(U5-AIN7/GPIO7-Pad6) -> /ADC_Group/Hall_Effect_Acquisition2/HE_Sensor_7
- U5 pad 7: unconnected-(U5-AVDD-Pad7) -> /ADC_Group/Hall_Effect_Acquisition2/3V3
- U5 pad 8: unconnected-(U5-DECAP-Pad8) -> /ADC_Group/Hall_Effect_Acquisition2/Decap
- U5 pad 9: unconnected-(U5-GND-Pad9) -> GND
- U6 pad 1: unconnected-(U6-AIN2/GPIO2-Pad1) -> /ADC_Group/Hall_Effect_Acquisition3/HE_Sensor_2
- U6 pad 10: unconnected-(U6-DVDD-Pad10) -> /ADC_Group/Hall_Effect_Acquisition3/3V3
- U6 pad 11: unconnected-(U6-ADDR-Pad11) -> /ADC_Group/Hall_Effect_Acquisition3/ADC_ADDR
- U6 pad 12: unconnected-(U6-ALERT-Pad12) -> /ADC3_ALERT
- U6 pad 13: unconnected-(U6-SCL-Pad13) -> /I2C_SCL_DAQ
- U6 pad 14: unconnected-(U6-SDA-Pad14) -> /I2C_SDA_DAQ
- U6 pad 15: unconnected-(U6-AIN0/GPIO0-Pad15) -> /ADC_Group/Hall_Effect_Acquisition3/HE_Sensor_0
- U6 pad 16: unconnected-(U6-AIN1/GPIO1-Pad16) -> /ADC_Group/Hall_Effect_Acquisition3/HE_Sensor_1
- U6 pad 17: unconnected-(U6-GND-Pad17) -> GND
- U6 pad 2: unconnected-(U6-AIN3/GPIO3-Pad2) -> /ADC_Group/Hall_Effect_Acquisition3/HE_Sensor_3
- U6 pad 3: unconnected-(U6-AIN4/GPIO4-Pad3) -> /ADC_Group/Hall_Effect_Acquisition3/HE_Sensor_4
- U6 pad 4: unconnected-(U6-AIN5/GPIO5-Pad4) -> /ADC_Group/Hall_Effect_Acquisition3/HE_Sensor_5
- U6 pad 5: unconnected-(U6-AIN6/GPIO6-Pad5) -> /ADC_Group/Hall_Effect_Acquisition3/HE_Sensor_6
- U6 pad 6: unconnected-(U6-AIN7/GPIO7-Pad6) -> /ADC_Group/Hall_Effect_Acquisition3/HE_Sensor_7
- U6 pad 7: unconnected-(U6-AVDD-Pad7) -> /ADC_Group/Hall_Effect_Acquisition3/3V3
- U6 pad 8: unconnected-(U6-DECAP-Pad8) -> /ADC_Group/Hall_Effect_Acquisition3/Decap
- U6 pad 9: unconnected-(U6-GND-Pad9) -> GND
- U7 pad 1: unconnected-(U7-AIN2/GPIO2-Pad1) -> /ADC_Group/Hall_Effect_Acquisition4/HE_Sensor_2
- U7 pad 10: unconnected-(U7-DVDD-Pad10) -> /ADC_Group/Hall_Effect_Acquisition4/3V3
- U7 pad 11: unconnected-(U7-ADDR-Pad11) -> /ADC_Group/Hall_Effect_Acquisition4/ADC_ADDR
- U7 pad 12: unconnected-(U7-ALERT-Pad12) -> /ADC4_ALERT
- U7 pad 13: unconnected-(U7-SCL-Pad13) -> /I2C_SCL_DAQ
- U7 pad 14: unconnected-(U7-SDA-Pad14) -> /I2C_SDA_DAQ
- U7 pad 15: unconnected-(U7-AIN0/GPIO0-Pad15) -> /ADC_Group/Hall_Effect_Acquisition4/HE_Sensor_0
- U7 pad 16: unconnected-(U7-AIN1/GPIO1-Pad16) -> /ADC_Group/Hall_Effect_Acquisition4/HE_Sensor_1
- U7 pad 17: unconnected-(U7-GND-Pad17) -> GND
- U7 pad 2: unconnected-(U7-AIN3/GPIO3-Pad2) -> /ADC_Group/Hall_Effect_Acquisition4/HE_Sensor_3
- U7 pad 3: unconnected-(U7-AIN4/GPIO4-Pad3) -> /ADC_Group/Hall_Effect_Acquisition4/HE_Sensor_4
- U7 pad 4: unconnected-(U7-AIN5/GPIO5-Pad4) -> /ADC_Group/Hall_Effect_Acquisition4/HE_Sensor_5
- U7 pad 5: unconnected-(U7-AIN6/GPIO6-Pad5) -> /ADC_Group/Hall_Effect_Acquisition4/HE_Sensor_6
- U7 pad 6: unconnected-(U7-AIN7/GPIO7-Pad6) -> /ADC_Group/Hall_Effect_Acquisition4/HE_Sensor_7
- U7 pad 7: unconnected-(U7-AVDD-Pad7) -> /ADC_Group/Hall_Effect_Acquisition4/3V3
- U7 pad 8: unconnected-(U7-DECAP-Pad8) -> /ADC_Group/Hall_Effect_Acquisition4/Decap
- U7 pad 9: unconnected-(U7-GND-Pad9) -> GND
- U8 pad 1: unconnected-(U8-AIN2/GPIO2-Pad1) -> /ADC_Group/Hall_Effect_Acquisition5/HE_Sensor_2
- U8 pad 10: unconnected-(U8-DVDD-Pad10) -> /ADC_Group/Hall_Effect_Acquisition5/3V3
- U8 pad 11: unconnected-(U8-ADDR-Pad11) -> /ADC_Group/Hall_Effect_Acquisition5/ADC_ADDR
- U8 pad 12: unconnected-(U8-ALERT-Pad12) -> /ADC5_ALERT
- U8 pad 13: unconnected-(U8-SCL-Pad13) -> /I2C_SCL_DAQ
- U8 pad 14: unconnected-(U8-SDA-Pad14) -> /I2C_SDA_DAQ
- U8 pad 15: unconnected-(U8-AIN0/GPIO0-Pad15) -> /ADC_Group/Hall_Effect_Acquisition5/HE_Sensor_0
- U8 pad 16: unconnected-(U8-AIN1/GPIO1-Pad16) -> /ADC_Group/Hall_Effect_Acquisition5/HE_Sensor_1
- U8 pad 17: unconnected-(U8-GND-Pad17) -> GND
- U8 pad 2: unconnected-(U8-AIN3/GPIO3-Pad2) -> /ADC_Group/Hall_Effect_Acquisition5/HE_Sensor_3
- U8 pad 3: unconnected-(U8-AIN4/GPIO4-Pad3) -> /ADC_Group/Hall_Effect_Acquisition5/HE_Sensor_4
- U8 pad 4: unconnected-(U8-AIN5/GPIO5-Pad4) -> /ADC_Group/Hall_Effect_Acquisition5/HE_Sensor_5
- U8 pad 5: unconnected-(U8-AIN6/GPIO6-Pad5) -> /ADC_Group/Hall_Effect_Acquisition5/HE_Sensor_6
- U8 pad 6: unconnected-(U8-AIN7/GPIO7-Pad6) -> /ADC_Group/Hall_Effect_Acquisition5/HE_Sensor_7
- U8 pad 7: unconnected-(U8-AVDD-Pad7) -> /ADC_Group/Hall_Effect_Acquisition5/3V3
- U8 pad 8: unconnected-(U8-DECAP-Pad8) -> /ADC_Group/Hall_Effect_Acquisition5/Decap
- U8 pad 9: unconnected-(U8-GND-Pad9) -> GND
- U9 pad 1: unconnected-(U9-AIN2/GPIO2-Pad1) -> /ADC_Group/Hall_Effect_Acquisition6/HE_Sensor_2
- U9 pad 10: unconnected-(U9-DVDD-Pad10) -> /ADC_Group/Hall_Effect_Acquisition6/3V3
- U9 pad 11: unconnected-(U9-ADDR-Pad11) -> /ADC_Group/Hall_Effect_Acquisition6/ADC_ADDR
- U9 pad 12: unconnected-(U9-ALERT-Pad12) -> /ADC6_ALERT
- U9 pad 13: unconnected-(U9-SCL-Pad13) -> /I2C_SCL_DAQ
- U9 pad 14: unconnected-(U9-SDA-Pad14) -> /I2C_SDA_DAQ
- U9 pad 15: unconnected-(U9-AIN0/GPIO0-Pad15) -> /ADC_Group/Hall_Effect_Acquisition6/HE_Sensor_0
- U9 pad 16: unconnected-(U9-AIN1/GPIO1-Pad16) -> /ADC_Group/Hall_Effect_Acquisition6/HE_Sensor_1
- U9 pad 17: unconnected-(U9-GND-Pad17) -> GND
- U9 pad 2: unconnected-(U9-AIN3/GPIO3-Pad2) -> /ADC_Group/Hall_Effect_Acquisition6/HE_Sensor_3
- U9 pad 3: unconnected-(U9-AIN4/GPIO4-Pad3) -> /ADC_Group/Hall_Effect_Acquisition6/HE_Sensor_4
- U9 pad 4: unconnected-(U9-AIN5/GPIO5-Pad4) -> /ADC_Group/Hall_Effect_Acquisition6/HE_Sensor_5
- U9 pad 5: unconnected-(U9-AIN6/GPIO6-Pad5) -> /ADC_Group/Hall_Effect_Acquisition6/HE_Sensor_6
- U9 pad 6: unconnected-(U9-AIN7/GPIO7-Pad6) -> /ADC_Group/Hall_Effect_Acquisition6/HE_Sensor_7
- U9 pad 7: unconnected-(U9-AVDD-Pad7) -> /ADC_Group/Hall_Effect_Acquisition6/3V3
- U9 pad 8: unconnected-(U9-DECAP-Pad8) -> /ADC_Group/Hall_Effect_Acquisition6/Decap
- U9 pad 9: unconnected-(U9-GND-Pad9) -> GND
Routing:
- added copper zone on B.Cu, net GND
- added copper zone on F.Cu, net GND

Commit message: PCB done
Parts:
- added G***: LOGO, Symbol:UIUC, F.Cu at (116.8, 143.2)
- added G***: LOGO, Symbol:horse, F.Cu at (134.0, 128.0)
- added J16: Conn_01x03_Pin, Connector_PinHeader_2.54mm:PinHeader_1x03_P2.54mm_Vertical, F.Cu at (116.5, 96.7)
- moved J5 138.5 mm to (94.5, 112.0), turned to 90 degrees
- moved SW2 137.4 mm to (102.2, 59.8)
- moved R42 133.6 mm to (149.4, 142.5), turned to 180 degrees
- moved R43 132.3 mm to (149.4, 140.8)
- moved R14 132.1 mm to (104.2, 120.5)
- moved R15 131.9 mm to (104.2, 122.2), turned to 180 degrees
- moved L1 131.0 mm to (104.2, 128.8)
- moved U1 127.6 mm to (104.2, 125.0)
- moved R8 126.0 mm to (101.8, 90.5), turned to -90 degrees
- moved R7 126.0 mm to (101.8, 87.0), turned to -90 degrees
- moved R9 125.6 mm to (103.5, 71.8)
- moved R10 125.6 mm to (103.5, 74.8), turned to 180 degrees
- moved R17 124.2 mm to (113.2, 130.5), turned to -90 degrees
- moved C3 123.5 mm to (101.0, 125.0), turned to 90 degrees
- moved J7 123.4 mm to (98.0, 85.4)
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Connections:
- net /5V renamed +5V
- C10 pad 2: /ADC_Group/Hall_Effect_Acquisition/3V3 -> +3V3
- C11 pad 2: /ADC_Group/Hall_Effect_Acquisition/3V3 -> +3V3
- C13 pad 2: /ADC_Group/Hall_Effect_Acquisition/3V3 -> +3V3
- C14 pad 2: /ADC_Group/Hall_Effect_Acquisition1/3V3 -> +3V3
- C15 pad 2: /ADC_Group/Hall_Effect_Acquisition1/3V3 -> +3V3
- C16 pad 2: /ADC_Group/Hall_Effect_Acquisition1/3V3 -> +3V3
- C18 pad 2: /ADC_Group/Hall_Effect_Acquisition1/3V3 -> +3V3
- C19 pad 2: /ADC_Group/Hall_Effect_Acquisition2/3V3 -> +3V3
- C20 pad 2: /ADC_Group/Hall_Effect_Acquisition2/3V3 -> +3V3
- C21 pad 2: /ADC_Group/Hall_Effect_Acquisition2/3V3 -> +3V3
- C23 pad 2: /ADC_Group/Hall_Effect_Acquisition2/3V3 -> +3V3
- C24 pad 2: /ADC_Group/Hall_Effect_Acquisition3/3V3 -> +3V3
- C25 pad 2: /ADC_Group/Hall_Effect_Acquisition3/3V3 -> +3V3
- C26 pad 2: /ADC_Group/Hall_Effect_Acquisition3/3V3 -> +3V3
- C28 pad 2: /ADC_Group/Hall_Effect_Acquisition3/3V3 -> +3V3
- C29 pad 2: /ADC_Group/Hall_Effect_Acquisition4/3V3 -> +3V3
- C30 pad 2: /ADC_Group/Hall_Effect_Acquisition4/3V3 -> +3V3
- C31 pad 2: /ADC_Group/Hall_Effect_Acquisition4/3V3 -> +3V3
- C33 pad 2: /ADC_Group/Hall_Effect_Acquisition4/3V3 -> +3V3
- C34 pad 2: /ADC_Group/Hall_Effect_Acquisition5/3V3 -> +3V3
- C35 pad 2: /ADC_Group/Hall_Effect_Acquisition5/3V3 -> +3V3
- C36 pad 2: /ADC_Group/Hall_Effect_Acquisition5/3V3 -> +3V3
- C38 pad 2: /ADC_Group/Hall_Effect_Acquisition5/3V3 -> +3V3
- C39 pad 2: /ADC_Group/Hall_Effect_Acquisition6/3V3 -> +3V3
- C40 pad 2: /ADC_Group/Hall_Effect_Acquisition6/3V3 -> +3V3
- C41 pad 2: /ADC_Group/Hall_Effect_Acquisition6/3V3 -> +3V3
- C43 pad 2: /ADC_Group/Hall_Effect_Acquisition6/3V3 -> +3V3
- C44 pad 2: /ADC_Group/Hall_Effect_Acquisition7/3V3 -> +3V3
- C45 pad 2: /ADC_Group/Hall_Effect_Acquisition7/3V3 -> +3V3
- C46 pad 2: /ADC_Group/Hall_Effect_Acquisition7/3V3 -> +3V3
- C48 pad 2: /ADC_Group/Hall_Effect_Acquisition7/3V3 -> +3V3
- C6 pad 2: /3V3 -> +3V3
- C8 pad 2: /3V3 -> +3V3
- C9 pad 2: /ADC_Group/Hall_Effect_Acquisition/3V3 -> +3V3
- J1 pad 1: /3V3 -> +3V3
- J10 pad 9: /ADC_Group/Hall_Effect_Acquisition2/3V3 -> +3V3
- J11 pad 9: /ADC_Group/Hall_Effect_Acquisition3/3V3 -> +3V3
- J12 pad 9: /ADC_Group/Hall_Effect_Acquisition4/3V3 -> +3V3
- J13 pad 9: /ADC_Group/Hall_Effect_Acquisition5/3V3 -> +3V3
- J14 pad 9: /ADC_Group/Hall_Effect_Acquisition6/3V3 -> +3V3
- J15 pad 9: /ADC_Group/Hall_Effect_Acquisition7/3V3 -> +3V3
- J6 pad 1: /3V3 -> +3V3
- J8 pad 9: /ADC_Group/Hall_Effect_Acquisition/3V3 -> +3V3
- J9 pad 9: /ADC_Group/Hall_Effect_Acquisition1/3V3 -> +3V3
- JP1 pad 3: /3V3 -> +3V3
- JP2 pad 2: /3V3 -> +3V3
- Q2 pad 2: /DTR -> /RTS
- R1 pad 1: /3V3 -> +3V3
- R18 pad 1: Net-(U2-IO48) -> Net-(U2-IO15)
- R2 pad 2: /3V3 -> +3V3
- R20 pad 2: /ADC_Group/Hall_Effect_Acquisition/3V3 -> +3V3
- R21 pad 2: /ADC_Group/Hall_Effect_Acquisition1/3V3 -> +3V3
- R22 pad 2: /ADC_Group/Hall_Effect_Acquisition2/3V3 -> +3V3
- R23 pad 2: /ADC_Group/Hall_Effect_Acquisition3/3V3 -> +3V3
- R24 pad 2: /ADC_Group/Hall_Effect_Acquisition4/3V3 -> +3V3
- R25 pad 2: /ADC_Group/Hall_Effect_Acquisition5/3V3 -> +3V3
- R26 pad 2: /ADC_Group/Hall_Effect_Acquisition6/3V3 -> +3V3
- R27 pad 2: /ADC_Group/Hall_Effect_Acquisition7/3V3 -> +3V3
- R3 pad 2: /3V3 -> +3V3
- R4 pad 1: /3V3 -> +3V3
- R5 pad 2: /3V3 -> +3V3
- R6 pad 2: /3V3 -> +3V3
- U10 pad 10: /ADC_Group/Hall_Effect_Acquisition7/3V3 -> +3V3
- U10 pad 7: /ADC_Group/Hall_Effect_Acquisition7/3V3 -> +3V3
- U2 pad 10: /SCR_DC -> /ADC6_ALERT
- U2 pad 11: /SCR_BLK -> /ADC7_ALERT
- U2 pad 12: /ADC4_ALERT -> /TCH_RST
- U2 pad 17: /ADC5_ALERT -> /SCR_INT
- U2 pad 18: /ADC6_ALERT -> /I2C_SDA_SCR
- U2 pad 19: /ADC7_ALERT -> /I2C_SCL_SCR
- U2 pad 2: /3V3 -> +3V3
- U2 pad 20: /I2C_SCL_DAQ -> /SCR_BLK
- U2 pad 21: /I2C_SDA_DAQ -> /SCR_DC
- U2 pad 22: /I2C_SCL_SCR -> /SCR_RST
- U2 pad 23: /SCR_INT -> /SCR_CS
- U2 pad 24: unconnected-(U2-IO47-Pad24) -> /SCR_MISO
- U2 pad 25: Net-(U2-IO48) -> /SCR_MOSI
- U2 pad 26: unconnected-(U2-IO45-Pad26) -> /SCR_SCLK
- U2 pad 31: /SCR_SCLK -> /I2C_SDA_DAQ
- U2 pad 32: /SCR_MOSI -> /I2C_SCL_DAQ
- U2 pad 33: /SCR_MISO -> /ADC4_ALERT
- U2 pad 34: /SCR_CS -> /ADC3_ALERT
- U2 pad 35: unconnected-(U2-IO42-Pad35) -> /ADC2_ALERT
- U2 pad 38: /TCH_RST -> /ADC1_ALERT
- U2 pad 39: /SCR_RST -> /ADC0_ALERT
- U2 pad 4: /ADC0_ALERT -> unconnected-(U2-IO4-Pad4)
- U2 pad 5: /ADC1_ALERT -> unconnected-(U2-IO5-Pad5)
- U2 pad 6: /ADC2_ALERT -> /LED_Driver
- U2 pad 7: /ADC3_ALERT -> unconnected-(U2-IO7-Pad7)
- U2 pad 8: /I2C_SDA_SCR -> Net-(U2-IO15)
- U2 pad 9: unconnected-(U2-IO16-Pad9) -> /ADC5_ALERT
- U3 pad 10: /ADC_Group/Hall_Effect_Acquisition/3V3 -> +3V3
- U3 pad 7: /ADC_Group/Hall_Effect_Acquisition/3V3 -> +3V3
- U4 pad 10: /ADC_Group/Hall_Effect_Acquisition1/3V3 -> +3V3
- U4 pad 7: /ADC_Group/Hall_Effect_Acquisition1/3V3 -> +3V3
- U5 pad 10: /ADC_Group/Hall_Effect_Acquisition2/3V3 -> +3V3
- U5 pad 7: /ADC_Group/Hall_Effect_Acquisition2/3V3 -> +3V3
- U6 pad 10: /ADC_Group/Hall_Effect_Acquisition3/3V3 -> +3V3
- U6 pad 7: /ADC_Group/Hall_Effect_Acquisition3/3V3 -> +3V3
- U7 pad 10: /ADC_Group/Hall_Effect_Acquisition4/3V3 -> +3V3
- U7 pad 7: /ADC_Group/Hall_Effect_Acquisition4/3V3 -> +3V3
- U8 pad 10: /ADC_Group/Hall_Effect_Acquisition5/3V3 -> +3V3
- U8 pad 7: /ADC_Group/Hall_Effect_Acquisition5/3V3 -> +3V3
- U9 pad 10: /ADC_Group/Hall_Effect_Acquisition6/3V3 -> +3V3
- U9 pad 7: /ADC_Group/Hall_Effect_Acquisition6/3V3 -> +3V3
Routing:
- net +3V3: track 0.00 -> 494.3 mm, vias 0 -> 37
- net /I2C_SDA_DAQ: track 0.00 -> 178.9 mm
- net /I2C_SCL_DAQ: track 0.00 -> 169.6 mm, vias 0 -> 14
- net +5V: track 0.00 -> 99.1 mm
- net /ADC6_ALERT: track 0.00 -> 96.8 mm, vias 0 -> 3
- net /ADC7_ALERT: track 0.00 -> 93.7 mm, vias 0 -> 3
- net /ADC5_ALERT: track 0.00 -> 87.0 mm, vias 0 -> 3
- net /ESP_BOOT: track 0.00 -> 80.8 mm, vias 0 -> 2
- net /TX: track 0.00 -> 72.9 mm, vias 0 -> 3
- net /RX: track 0.00 -> 72.2 mm, vias 0 -> 3
- net /ADC4_ALERT: track 0.00 -> 62.7 mm, vias 0 -> 3
- net /ADC3_ALERT: track 0.00 -> 52.6 mm, vias 0 -> 3
- net /ESP_EN: track 0.00 -> 50.3 mm, vias 0 -> 2
- net /LED_Driver: track 0.00 -> 48.7 mm, vias 0 -> 2
- net /ADC2_ALERT: track 0.00 -> 42.7 mm, vias 0 -> 3
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Other:
- board text added: "3V3"
- board text added: "3V3 ON!"
- board text added: "5V"
- board text added: "A1"
- board text added: "A2"
- board text added: "A3"
- board text added: "A4"
- board text added: "A5"
- board text added: "A6"
- board text added: "A7"
- board text added: "A8"
- board text added: "B1"
- board text added: "B2"
- board text added: "B3"
- board text added: "B4"
- board text added: "B5"
- board text added: "B6"
- board text added: "B7"
- board text added: "B8"
- board text added: "BOOT"
- board text added: "C1"
- board text added: "C2"
- board text added: "C3"
- board text added: "C4"
- board text added: "C5"
- board text added: "C6"
- board text added: "C7"
- board text added: "C8"
- board text added: "D1"
- board text added: "D2"
- board text added: "D3"
- board text added: "D4"
- board text added: "D5"
- board text added: "D6"
- board text added: "D7"
- board text added: "D8"
- board text added: "DO NO CONNECT BEFORE TESTING"
- board text added: "DTR"
- board text added: "Display Header"
- board text added: "E1"
- board text added: "E2"
- board text added: "E3"
- board text added: "E4"
- board text added: "E5"
- board text added: "E6"
- board text added: "E7"
- board text added: "E8"
- board text added: "En Passant"
- board text added: "F1"
- board text added: "F2"
- board text added: "F3"
- board text added: "F4"
- board text added: "F5"
- board text added: "F6"
- board text added: "F7"
- board text added: "F8"
- board text added: "G1"
- board text added: "G2"
- board text added: "G3"
- board text added: "G4"
- board text added: "G5"
- board text added: "G6"
- board text added: "G7"
- board text added: "G8"
- board text added: "GND"
- board text added: "H1"
- board text added: "H2"
- board text added: "H3"
- board text added: "H4"
- board text added: "H5"
- board text added: "H6"
- board text added: "H7"
- board text added: "H8"
- board text added: "LED Header"
- board text added: "LED_Driver"
- board text added: "Networked Chess Main PCB ECE 445 Team-51"
- board text added: "Quinn Athas Danny Guller Payton Schutte"
- board text added: "RESET"
- board text added: "RST"
- board text added: "RX"
- board text added: "SCL_SCR"
- board text added: "SCR_BLK"
- board text added: "SCR_CLK"
- board text added: "SCR_CS"
- board text added: "SCR_DC"
- board text added: "SCR_INT"
- board text added: "SCR_MISO"
- board text added: "SCR_MOSI"
- board text added: "SCR_RST"
- board text added: "SDA_SCR"
- board text added: "TCH_RST"
- board text added: "TX"
- board text added: "UART Prog Header"
- board text added: "this is where the code goes"
