File: ECE-445-PCBs/Main_Board/Main_Board_PCB.kicad_sch (KiCad schematic)
At the start: 5 parts, among them J1 USB_C_Receptacle_USB2.0_16P, J2 Screw_Terminal_01x08, J3 Conn_01x02_Pin, U1 ESP32-S3-WROOM-1, U2 TLV62569DDC

Commit message: PSU done
Parts:
- added C41, C42, C43: 10uF, symbol Device:C
- added C44: 4.7uF, symbol Device:C
- added L1: 2.2uH, symbol Device:L
- added R1, R2: 5.1k, symbol Device:R_US
- added R10, R19: 33k, symbol Device:R_US
- added R11, R13, R14, R15, R16, R18, R20, R6, R9: R_US, symbol Device:R_US
- added R12, R21, R4: 100k, symbol Device:R_US
- added R17, R8: 11k, symbol Device:R_US
- added R3: 442k, symbol Device:R_US
- added R5: 475k, symbol Device:R_US
- added R7: 0, symbol Device:R_US
Connections:
- net Hall_Effect_Acquisition/ADC_ADDR: now also R6.1, R7.2
- net Hall_Effect_Acquisition1/ADC_ADDR: now also R8.2, R9.1
- net Hall_Effect_Acquisition2/ADC_ADDR: now also R10.2, R11.1
- net Hall_Effect_Acquisition3/ADC_ADDR: now also R12.2, R13.1
- net Hall_Effect_Acquisition4/ADC_ADDR: now also R14.2, R15.1
- net Hall_Effect_Acquisition5/ADC_ADDR: now also R16.2, R17.1
- net Hall_Effect_Acquisition6/ADC_ADDR: now also R18.2, R19.1
- net Hall_Effect_Acquisition7/ADC_ADDR: now also R20.2, R21.1
- net GND: now reaches U1.1 (GND), U1.40 (GND), U1.41 (GND)
- net GND: now also J1.A1 (GND), J1.A12 (GND), J1.B1 (GND), J1.B12 (GND), U2.2 (GND), C41.1, C42.1, C43.1, C44.1, R1.2, R11.2, R13.2, R15.2, R17.2, R19.2, R2.1, R21.2, R4.2, R6.2, R9.2
- net USB_D_N: now reaches U1.13 (USB_D-)
- net USB_D_N: now also J1.A7 (D-), J1.B7 (D-)
- net USB_D_P: now reaches U1.14 (USB_D+)
- net USB_D_P: now also J1.A6 (D+), J1.B6 (D+)
- net 3V3: now reaches U1.2 (3V3)
- net 3V3: now also U1.3 (EN), C41.2, C42.2, C43.2, L1.2, R3.1
- net 5V: now reaches J1.A4 (VBUS), J1.A9 (VBUS), J1.B4 (VBUS), J1.B9 (VBUS)
- net 5V: now also U2.1 (EN), U2.4 (VIN), C44.2, R5.2
- net at J1.A5 (CC1): now also R1.1
- net at J1.B5 (CC2): now also R2.2
- net at U2.3 (SW): now also L1.1
- net at U2.5 (PG): now also R5.1
- net at U2.6 (FB): now also R3.2, R4.1
- new net Hall_Effect_Acquisition/Decap: R7.1
- new net Hall_Effect_Acquisition1/Decap: R8.1
- new net Hall_Effect_Acquisition2/Decap: R10.1
- new net Hall_Effect_Acquisition3/Decap: R12.1
- new net Hall_Effect_Acquisition4/Decap: R14.1
- new net Hall_Effect_Acquisition5/Decap: R16.1
- new net Hall_Effect_Acquisition6/Decap: R18.1
- new net Hall_Effect_Acquisition7/Decap: R20.1
- no-connect marks 0 -> 3
Other:
- sheet Hall_Effect_Acquisition ports: added Decap; removed none
- sheet Hall_Effect_Acquisition1 ports: added Decap; removed none
- sheet Hall_Effect_Acquisition2 ports: added Decap; removed none
- sheet Hall_Effect_Acquisition3 ports: added Decap; removed none
- sheet Hall_Effect_Acquisition4 ports: added Decap; removed none
- sheet Hall_Effect_Acquisition5 ports: added Decap; removed none
- sheet Hall_Effect_Acquisition6 ports: added Decap; removed none
- sheet Hall_Effect_Acquisition7 ports: added Decap; removed none
- note added: "ADDR: 0x10h"
- note added: "ADDR: 0x11h"
- note added: "ADDR: 0x12h"
- note added: "ADDR: 0x13h"
- note added: "ADDR: 0x14h"
- note added: "ADDR: 0x15h"
- note added: "ADDR: 0x16h"
- note added: "ADDR: 0x17h"
- moved on the sheet: J1, J2, J3, U1, U2

Commit message: ESP setup done
Parts:
- added C45, C46: 1uF, symbol Device:C
- added C47: 0.1uF, symbol Device:C
- added C48: 22uF, symbol Device:C
- added R22, R23: 10k, symbol Device:R_US
- added SW1, SW2: SW_Push, symbol Switch:SW_Push
Connections:
- net 3V3: now also C47.2, C48.2, R22.1, R23.1; no longer U1.3 (EN)
- net GND: now also C45.2, C46.2, C47.1, C48.1, SW1.2, SW2.2
- net I2C_SCL_Display: now reaches U1.12 (IO8)
- net I2C_SDA_Display: now reaches U1.17 (IO9)
- net ESP_BOOT: now reaches U1.27 (IO0)
- net ESP_BOOT: now also C46.1, R23.2, SW2.1
- net I2C_SCL_Board: now reaches U1.4 (IO4)
- net I2C_SDA_Board: now reaches U1.5 (IO5)
- new net ESP_EN: C45.1, R22.2, SW1.1, U1.3 (EN)
- no-connect marks 3 -> 8
Other:
- note added: "BOOT"
- note added: "IO45 left to default 0 for 3.3V SPI"
- note added: "IO46 left to default 0 for boot mode"
- note added: "RESET"
- moved on the sheet: U1

Commit message: started placement
Parts:
- removed J2: Screw_Terminal_01x08, TerminalBlock:OSTVN08A150, symbol Connector:Screw_Terminal_01x08
- removed R10: 33k, symbol Device:R_US
- removed R13, R14, R15, R20, R9: R_US, symbol Device:R_US
- removed R21: 100k, symbol Device:R_US
- added D1, D2: RED LED, LED_SMD:LED_0603_1608Metric, symbol Device:LED
- added H1, H2, H3, H4: MountingHole_Pad, MountingHole:MountingHole_3.2mm_M3_DIN965_Pad, symbol Mechanical:MountingHole_Pad
- added J1: Conn_01x14_Pin, Connector_PinHeader_2.54mm:PinHeader_1x14_P2.54mm_Vertical, symbol Connector:Conn_01x14_Pin
- added J2, J5, J6: Conn_01x02_Pin, Connector_PinHeader_2.54mm:PinHeader_1x02_P2.54mm_Vertical, symbol Connector:Conn_01x02_Pin
- added J7: Conn_01x05_Pin, Connector_PinHeader_2.54mm:PinHeader_1x05_P2.54mm_Vertical, symbol Connector:Conn_01x05_Pin
- added JP1: SolderJumper_3_Open, Jumper:SolderJumper-3_P1.3mm_Open_Pad1.0x1.5mm, symbol Jumper:SolderJumper_3_Open
- added JP2: SolderJumper_2_Open, Jumper:SolderJumper-2_P1.3mm_Open_Pad1.0x1.5mm, symbol Jumper:SolderJumper_2_Open
- added Q1, Q2: SS8050, Package_TO_SOT_SMD:SOT-23, symbol Transistor_BJT:SS8050
- added R2, R3, R5: 4.7k, Resistor_SMD:R_0603_1608Metric, symbol Device:R_US
- C1: renamed from C45; footprint (none) -> Capacitor_SMD:C_0603_1608Metric
- C2: renamed from C46; footprint (none) -> Capacitor_SMD:C_0603_1608Metric
- C3: renamed from C44; footprint (none) -> Capacitor_SMD:C_0603_1608Metric
- C4: renamed from C41; footprint (none) -> Capacitor_SMD:C_0603_1608Metric
- C5: renamed from C42; footprint (none) -> Capacitor_SMD:C_0603_1608Metric
- C6: renamed from C48; footprint (none) -> Capacitor_SMD:C_0603_1608Metric
- C7: renamed from C43; footprint (none) -> Capacitor_SMD:C_0603_1608Metric
- C8: renamed from C47; footprint (none) -> Capacitor_SMD:C_0603_1608Metric
- J3: footprint Connector_Harwin:HARWIN_M20-9990246 -> Connector_PinHeader_2.54mm:PinHeader_1x02_P2.54mm_Vertical
- L1: footprint (none) -> Inductor_SMD:L_Coilcraft_1008HQ_2520Metric
- R1: renamed from R22; value 10k -> 100k; footprint (none) -> Resistor_SMD:R_0603_1608Metric
- R10: renamed from R2; footprint (none) -> Resistor_SMD:R_0603_1608Metric
- R11: value R_US -> 10k; footprint (none) -> Resistor_SMD:R_0603_1608Metric; now fitted
- R12: value 100k -> 10k; footprint (none) -> Resistor_SMD:R_0603_1608Metric
- R13: renamed from R5; footprint (none) -> Resistor_SMD:R_0603_1608Metric
- R14: renamed from R3; value 442k -> 450k; footprint (none) -> Resistor_SMD:R_0603_1608Metric
- R15: renamed from R4; footprint (none) -> Resistor_SMD:R_0603_1608Metric
- R16: value R_US -> 1k; footprint (none) -> Resistor_SMD:R_0603_1608Metric; now fitted
- R17: value 11k -> 470; footprint (none) -> Resistor_SMD:R_0603_1608Metric
- R18: value R_US -> 470; footprint (none) -> Resistor_SMD:R_0603_1608Metric; now fitted
- R19: value 33k -> 1k; footprint (none) -> Resistor_SMD:R_0603_1608Metric; now not fitted
- R4: renamed from R23; value 10k -> 100k; footprint (none) -> Resistor_SMD:R_0603_1608Metric
- R6: value R_US -> 4.7k; footprint (none) -> Resistor_SMD:R_0603_1608Metric; now fitted
- R7: value 0 -> 10k; footprint (none) -> Resistor_SMD:R_0603_1608Metric
- R8: value 11k -> 10k; footprint (none) -> Resistor_SMD:R_0603_1608Metric
- R9: renamed from R1; footprint (none) -> Resistor_SMD:R_0603_1608Metric
- SW1, SW2: footprint (none) -> Button_Switch_THT:SW_TH_Tactile_Omron_B3F-100x
- renumbered J1 to J4, U2 to U1, U1 to U2
Connections:
- net Hall_Effect_Acquisition3/ADC_ADDR is gone; now on net ESP_BOOT: R12.2
- net Hall_Effect_Acquisition6/Decap is gone; now on an unnamed net: R18.1
- net 3V3: now also R19.2, R6.2, J1.1 (Pin_1), J6.1 (Pin_1), JP1.3 (B), JP2.2 (B), R2.2, R3.2, R5.2; no longer C4.2, C5.2, C7.2, L1.2, R14.1
- net 5V: now also J5.1 (Pin_1)
- net ESP_EN: now also R11.2
- net GND: now also D1.1 (K), D2.1 (K), H1.1, H2.1, H3.1, H4.1, J1.13 (Pin_13), J1.2 (Pin_2), J5.2 (Pin_2), J6.2 (Pin_2), J7.5 (Pin_5), JP1.1 (A); no longer R11.2, R17.2, R19.2, R6.2
- net SCR_DC: now reaches U2.10 (IO17)
- net SCR_DC: now also J1.8 (Pin_8)
- net SCR_BLK: now reaches U2.11 (IO18)
- net SCR_BLK: now also J1.9 (Pin_9)
- net at U2.15 (IO3): now also R16.2
- net at U2.16 (IO46): now also R19.1
- net ADC6_ALERT: now reaches U2.18 (IO10)
- net ADC7_ALERT: now reaches U2.19 (IO11)
- net I2C_SCL_DAQ: now reaches U2.20 (IO12)
- net I2C_SCL_DAQ: now also J2.2 (Pin_2), R2.1
- net I2C_SDA_DAQ: now reaches U2.21 (IO13)
- net I2C_SDA_DAQ: now also J2.1 (Pin_1), R3.1
- net I2C_SCL_SCR: now reaches U2.22 (IO14)
- net I2C_SCL_SCR: now also J3.1 (Pin_1), R6.1, J1.10 (Pin_10)
- net SCR_INT: now reaches U2.23 (IO21)
- net SCR_INT: now also J1.12 (Pin_12)
- net SCR_SCLK: now reaches U2.31 (IO38)
- net SCR_SCLK: now also J1.3 (Pin_3)
- net SCR_MOSI: now reaches U2.32 (IO39)
- net SCR_MOSI: now also J1.4 (Pin_4)
- net SCR_MISO: now reaches U2.33 (IO40)
- net SCR_MISO: now also J1.5 (Pin_5)
- net SCR_CS: now reaches U2.34 (IO41)
- net SCR_CS: now also J1.6 (Pin_6)
- net RX: now reaches U2.36 (RXD0)
- net RX: now also J7.4 (Pin_4)
- net TX: now reaches U2.37 (TXD0)
- net TX: now also J7.3 (Pin_3)
- net TCH_RST: now reaches U2.38 (IO2)
- net TCH_RST: now also J1.14 (Pin_14)
- net SCR_RST: now reaches U2.39 (IO1)
- net SCR_RST: now also J1.7 (Pin_7)
- net ADC2_ALERT: now reaches U2.6 (IO6)
- net ADC3_ALERT: now reaches U2.7 (IO7)
- net I2C_SDA_SCR: now reaches U2.8 (IO15)
- net I2C_SDA_SCR: now also J3.2 (Pin_2), J1.11 (Pin_11), R5.1
- net Hall_Effect_Acquisition/ADC_ADDR: no longer names the net of R7.2
- net Hall_Effect_Acquisition/ADC_ADDR: now also Q1.1 (B); no longer R6.1
- net Hall_Effect_Acquisition/Decap renamed RTS
- net RTS: now also J7.1 (Pin_1)
- net Hall_Effect_Acquisition1/ADC_ADDR: no longer names the net of R8.2
- net Hall_Effect_Acquisition1/ADC_ADDR: now also Q2.1 (B)
- net Hall_Effect_Acquisition1/Decap renamed DTR
- net DTR: now also J7.2 (Pin_2), Q1.2 (E), Q2.2 (E)
- net Hall_Effect_Acquisition2/ADC_ADDR: no longer names the net of R11.1
- net Hall_Effect_Acquisition2/ADC_ADDR: now also Q1.3 (C)
- net Hall_Effect_Acquisition3/Decap: no longer names the net of R12.1
- net Hall_Effect_Acquisition3/Decap: now also Q2.3 (C)
- net Hall_Effect_Acquisition5/ADC_ADDR: no longer names the net of R17.1
- net Hall_Effect_Acquisition5/ADC_ADDR: now also C4.2, C5.2, C7.2, L1.2, R14.1, JP2.1 (A); no longer R16.2
- net Hall_Effect_Acquisition5/Decap: no longer names the net of R16.1
- net Hall_Effect_Acquisition5/Decap: now also JP1.2 (C)
- net Hall_Effect_Acquisition6/ADC_ADDR: no longer names the net of R18.2
- net Hall_Effect_Acquisition6/ADC_ADDR: now also D2.2 (A); no longer R19.1
- net I2C_SCL_Board renamed ADC0_ALERT
- net I2C_SCL_Display renamed ADC4_ALERT
- net I2C_SDA_Board renamed ADC1_ALERT
- net I2C_SDA_Display renamed ADC5_ALERT
- new net: D1.2 (A), R17.2
- no-connect marks 8 -> 10
Other:
- removed sheet Hall_Effect_Acquisition
- removed sheet Hall_Effect_Acquisition1
- removed sheet Hall_Effect_Acquisition2
- removed sheet Hall_Effect_Acquisition3
- removed sheet Hall_Effect_Acquisition4
- removed sheet Hall_Effect_Acquisition5
- removed sheet Hall_Effect_Acquisition6
- removed sheet Hall_Effect_Acquisition7
- added sheet ADC_Group (ADC_Group.kicad_sch)
- note added: "UART PROG"
- note removed: "ADDR: 0x10h"
- note removed: "ADDR: 0x11h"
- note removed: "ADDR: 0x12h"
- note removed: "ADDR: 0x13h"
- note removed: "ADDR: 0x14h"
- note removed: "ADDR: 0x15h"
- note removed: "ADDR: 0x16h"
- note removed: "ADDR: 0x17h"
- note removed: "IO45 left to default 0 for 3.3V SPI"
- note removed: "IO46 left to default 0 for boot mode"
- moved on the sheet: C3, C4, C5, C7, J4, L1, R10, R13, R14, R15, R9, U1

Commit message: PCB done
Parts:
- added J16: Conn_01x03_Pin, Connector_PinHeader_2.54mm:PinHeader_1x03_P2.54mm_Vertical, symbol Connector:Conn_01x03_Pin
- J4: footprint Connector_USB:USB4215-03-A -> Connector_USB:USB_C_Receptacle_G-Switch_GT-USB-7010ASV
Connections:
- net 3V3: no longer C6.2, C8.2, J1.1 (Pin_1), J6.1 (Pin_1), JP1.3 (B), JP2.2 (B), R1.1, R2.2, R3.2, R4.1, R5.2, R6.2, U2.2 (3V3)
- net ADC0_ALERT: now also U2.39 (IO1); no longer U2.4 (IO4)
- net ADC1_ALERT: now also U2.38 (IO2); no longer U2.5 (IO5)
- net ADC2_ALERT: now also U2.35 (IO42); no longer U2.6 (IO6)
- net ADC3_ALERT: now also U2.34 (IO41); no longer U2.7 (IO7)
- net ADC4_ALERT: now also U2.33 (IO40); no longer U2.12 (IO8)
- net ADC5_ALERT: now also U2.9 (IO16); no longer U2.17 (IO9)
- net ADC6_ALERT: now also U2.10 (IO17); no longer U2.18 (IO10)
- net ADC7_ALERT: now also U2.11 (IO18); no longer U2.19 (IO11)
- net DTR: no longer Q2.2 (E)
- net GND: now also J16.3 (Pin_3)
- net I2C_SCL_DAQ: now also U2.32 (IO39); no longer U2.20 (IO12)
- net I2C_SCL_SCR: now also U2.19 (IO11); no longer U2.22 (IO14)
- net I2C_SDA_DAQ: now also U2.31 (IO38); no longer U2.21 (IO13)
- net I2C_SDA_SCR: now also U2.18 (IO10); no longer U2.8 (IO15)
- net RTS: now also Q2.2 (E)
- net SCR_BLK: now also U2.20 (IO12); no longer U2.11 (IO18)
- net SCR_CS: now also U2.23 (IO21); no longer U2.34 (IO41)
- net SCR_DC: now also U2.21 (IO13); no longer U2.10 (IO17)
- net SCR_INT: now also U2.17 (IO9); no longer U2.23 (IO21)
- net SCR_MISO: now also U2.24 (IO47); no longer U2.33 (IO40)
- net SCR_MOSI: now also U2.25 (IO48); no longer U2.32 (IO39)
- net SCR_RST: now also U2.22 (IO14); no longer U2.39 (IO1)
- net SCR_SCLK: now also U2.26 (IO45); no longer U2.31 (IO38)
- net TCH_RST: now also U2.12 (IO8); no longer U2.38 (IO2)
- net at R18.1: now also U2.8 (IO15); no longer U2.25 (IO48)
- net 5V renamed +5V
- net +5V: now also J16.1 (Pin_1)
- new net +3V3: C6.2, C8.2, J1.1 (Pin_1), J6.1 (Pin_1), JP1.3 (B), JP2.2 (B), R1.1, R2.2, R3.2, R4.1, R5.2, R6.2, U2.2 (3V3)
- new net LED_Driver: J16.2 (Pin_2), U2.6 (IO6)
- no-connect marks 10 -> 9
Other:
- moved on the sheet: D2, R18, R19
