File: ECE-445-PCBs/Main_Board/Hall_Effect_Acquisition.kicad_sch (KiCad schematic)
At the start: 7 parts, among them J4 Conn_02x05_Odd_Even, U9 ADS7128IRTER

Commit message: PSU done
Connections:
- net Decap: now reaches C3.2, U9.8 (DECAP)

Commit message: started placement
Parts:
- added R20: 4.7k, Resistor_SMD:R_0603_1608Metric, symbol Device:R_US
- C10: renamed from C2; footprint (none) -> Capacitor_SMD:C_0603_1608Metric
- C11: renamed from C5; footprint (none) -> Capacitor_SMD:C_0603_1608Metric
- C12: renamed from C3; footprint (none) -> Capacitor_SMD:C_0603_1608Metric
- C13: renamed from C4; footprint (none) -> Capacitor_SMD:C_0603_1608Metric
- C9: renamed from C1; footprint (none) -> Capacitor_SMD:C_0603_1608Metric
- renumbered J4 to J8, U9 to U3
Connections:
- net 3V3: now also R20.2
- net ADC_ALERT: now also R20.1

Commit message: PCB done
Connections:
- net 3V3 renamed +3V3

Commit message: BOM csv added
Parts:
- C10, C11, C12, C13: now in the parts list
Changed lines of the file:
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@@
 		(unit 1)
 		(exclude_from_sim no)
-		(in_bom no)
+		(in_bom yes)
 		(on_board yes)
 		(dnp no)
@@
 		(unit 1)
 		(exclude_from_sim no)
-		(in_bom no)
+		(in_bom yes)
 		(on_board yes)
 		(dnp no)
@@
 		(unit 1)
 		(exclude_from_sim no)
-		(in_bom no)
+		(in_bom yes)
 		(on_board yes)
 		(dnp no)
@@
 		(unit 1)
 		(exclude_from_sim no)
-		(in_bom no)
-		(on_board yes)
-		(dnp no)
+		(in_bom yes)
+		(on_board yes)
+		(dnp no)
